File: RP2040_DevBoard_LiPo.kicad_pcb (KiCad board)
At the start: 2 copper layers, 24 x 48 mm, 56 parts, among them J1 USB_C_Receptacle_USB2.0, J2 Conn_01x18, J3 Battery, J4 Conn_01x18, Q1 DMP2045U, SW1 SW_Push, SW2 SW_Push, SW3 Vin_Switch, U1 W25Q128JVS, U2 USBLC6-2SC6, U3 SOT23-5 200mA 3.3V, U4 RP2040, U5 MCP73831-2-OT, Y1 Crystal_GND23

Commit message: Updated Schematic. Added LCSC part for most parts
Parts:
- removed C1: 100 nF, Diode_SMD:D_0603_1608Metric
- removed C10, C12, C13, C14, C15, C17, C18, C19, C20, C5, C6, C7, C9: 1uF, Capacitor_SMD:C_0603_1608Metric
- removed C11, C8: 1u, Capacitor_SMD:C_0603_1608Metric
- removed C16, C21: 4u7, Capacitor_SMD:C_0603_1608Metric
- removed C2, C3: 22pF, Capacitor_SMD:C_0603_1608Metric
- removed C4: 10uF, Capacitor_SMD:C_0603_1608Metric
- removed D1: BSD3C051V, Diode_SMD:D_SOD-323
- removed D2: LED, LED_SMD:LED_0603_1608Metric
- removed D3: D_Schottky, Diode_SMD:D_0603_1608Metric
- removed D4: LED, LED_SMD:LED_0805_2012Metric_Pad1.15x1.40mm_HandSolder
- removed F1: 750 mA, Fuse:Fuse_0603_1608Metric
- removed J1: USB_C_Receptacle_USB2.0, Connector_USB:USB_C_Receptacle_HRO_TYPE-C-31-M-12
- removed J2, J4: Conn_01x18, Connector_PinSocket_2.54mm:PinSocket_1x18_P2.54mm_Vertical
- removed J3: Battery, Connector_JST:JST_PH_S2B-PH-SM4-TB_1x02-1MP_P2.00mm_Horizontal
- removed L1, L2: BLM15PX121SN1D, Inductor_SMD:L_0603_1608Metric
- removed Q1: DMP2045U, Package_TO_SOT_SMD:SOT-23
- removed R1: 1 MOhm, Resistor_SMD:R_0603_1608Metric
- removed R10, R2, R3, R7: 1k, Resistor_SMD:R_0603_1608Metric
- removed R11, R12: 27, Resistor_SMD:R_0603_1608Metric
- removed R13, R6: 470, Resistor_SMD:R_0603_1608Metric
- removed R14: 2k, Resistor_SMD:R_0603_1608Metric
- removed R4, R5: 5k1, Resistor_SMD:R_0603_1608Metric
- removed R8, R9: 10k, Resistor_SMD:R_0603_1608Metric
- removed SW1, SW2: SW_Push, Button_Switch_SMD:SW_Push_SPST_NO_Alps_SKRK
- removed SW3: Vin_Switch, Buggy_Footprints:switch123
- removed U1: W25Q128JVS, Package_SO:SOIC-8_5.23x5.23mm_P1.27mm
- removed U2: USBLC6-2SC6, Package_TO_SOT_SMD:SOT-23-6
- removed U3: SOT23-5 200mA 3.3V, Package_TO_SOT_SMD:SOT-23-5
- removed U4: RP2040, Package_DFN_QFN:QFN-56-1EP_7x7mm_P0.4mm_EP3.2x3.2mm
- removed U5: MCP73831-2-OT, Package_TO_SOT_SMD:SOT-23-5
- removed Y1: Crystal_GND23, Crystal:Crystal_SMD_3225-4Pin_3.2x2.5mm
Other:
- board outline removed

Commit message: started routing
Parts:
- added C1: 100nF, Capacitor_SMD:C_0402_1005Metric, F.Cu at (185.6, 27.6)
- added C10: 22pF, Capacitor_SMD:C_0402_1005Metric, F.Cu at (187.3, 71.9)
- added C11: 22pF, Capacitor_SMD:C_0402_1005Metric, F.Cu at (187.6, 70.5)
- added C12: 1u, Capacitor_SMD:C_0402_1005Metric, F.Cu at (153.0, 107.0)
- added C13: 100nF, Capacitor_SMD:C_0402_1005Metric, F.Cu at (157.0, 107.0)
- added C14: 100nF, Capacitor_SMD:C_0402_1005Metric, F.Cu at (160.5, 107.0)
- added C15: 1u, Capacitor_SMD:C_0402_1005Metric, F.Cu at (178.0, 92.0)
- added C16: 100nF, Capacitor_SMD:C_0402_1005Metric, F.Cu at (174.5, 105.0)
- added C17: 100nF, Capacitor_SMD:C_0402_1005Metric, F.Cu at (183.5, 94.0)
- added C18: 100nF, Capacitor_SMD:C_0402_1005Metric, F.Cu at (170.5, 101.0)
- added C19: 100nF, Capacitor_SMD:C_0402_1005Metric, F.Cu at (175.5, 100.9)
- added C2: 10uF, Capacitor_SMD:C_0402_1005Metric, F.Cu at (188.1, 26.6)
- added C20: 100nF, Capacitor_SMD:C_0402_1005Metric, F.Cu at (178.5, 97.0)
- added C21: 100nF, Capacitor_SMD:C_0402_1005Metric, F.Cu at (180.0, 104.0)
- added C22: 100nF, Capacitor_SMD:C_0402_1005Metric, F.Cu at (182.5, 100.0)
- added C3: 100nF, Capacitor_SMD:C_0402_1005Metric, F.Cu at (137.4, 94.4)
- added C4: 1u, Capacitor_SMD:C_0402_1005Metric, F.Cu at (184.3, 45.8)
- added C5: 1u, Capacitor_SMD:C_0402_1005Metric, F.Cu at (182.8, 43.6)
- added C6: 100nF, Capacitor_SMD:C_0402_1005Metric, F.Cu at (187.4, 45.2)
- added C7: 10 uF, Capacitor_SMD:CP_Elec_3x5.3, F.Cu at (175.3, 39.7)
- added C8: 4.7 uF, Capacitor_SMD:C_0402_1005Metric, F.Cu at (173.6, 41.7)
- added C9: 10 uF, Capacitor_SMD:CP_Elec_3x5.3, F.Cu at (175.0, 45.9)
- added D1: BSD3C051V, Diode_SMD:D_SOD-323, F.Cu at (186.2, 30.3)
- added D3: D_Schottky, Diode_SMD:D_SOD-323, F.Cu at (179.1, 40.2)
- added D4: LED, LED_SMD:LED_1206_3216Metric, F.Cu at (169.8, 25.6)
- added F1: 750 mA, Fuse:Fuse_0603_1608Metric, F.Cu at (188.7, 25.1)
- added J1: HRO_TYPE-C-31-M-14, Connector_USB:USB_C_Receptacle_HRO_TYPE-C-31-M-12, F.Cu at (179.0, 28.0)
- added J2: Conn_01x18, Connector_PinSocket_2.54mm:PinSocket_1x18_P2.54mm_Vertical, F.Cu at (90.0, 42.0)
- added J3: Conn_01x18, Connector_PinSocket_2.54mm:PinSocket_1x18_P2.54mm_Vertical, F.Cu at (76.0, 43.0)
- added J4: Battery, Connector_JST:JST_EH_S2B-EH_1x02_P2.50mm_Horizontal, F.Cu at (170.9, 45.8)
- added L1: BLM15PX121SN1D, Inductor_SMD:L_0402_1005Metric, F.Cu at (185.6, 28.7)
- added L2: BLM15PX121SN1D, Inductor_SMD:L_0402_1005Metric, F.Cu at (185.8, 24.9)
- added Q1: DMP2045U, Package_TO_SOT_SMD:SOT-23, F.Cu at (178.6, 42.9)
- added R1: 1 MOhm, Resistor_SMD:R_0402_1005Metric, F.Cu at (185.6, 26.5)
- added R10: 1.5k, Resistor_SMD:R_0402_1005Metric, F.Cu at (168.8, 27.4)
- added R11: 5k, Resistor_SMD:R_0603_1608Metric, F.Cu at (174.7, 35.2)
- added R12: 1k, Resistor_SMD:R_0402_1005Metric, F.Cu at (187.5, 68.9)
- added R13: 27, Resistor_SMD:R_0402_1005Metric, F.Cu at (178.4, 68.8)
- added R14: 27, Resistor_SMD:R_0402_1005Metric, F.Cu at (177.1, 68.8)
- added R2: 5k1, Resistor_SMD:R_0402_1005Metric, F.Cu at (181.5, 34.8)
- added R3: 5k1, Resistor_SMD:R_0402_1005Metric, F.Cu at (176.5, 34.8)
- added R5: 1k, Resistor_SMD:R_0402_1005Metric, F.Cu at (137.4, 92.3)
- added R6: 1k, Resistor_SMD:R_0402_1005Metric, F.Cu at (125.0, 79.0)
- added R7: 1.5k, Resistor_SMD:R_0402_1005Metric, F.Cu at (181.5, 40.2)
- added R8: 10k, Resistor_SMD:R_0402_1005Metric, F.Cu at (185.3, 43.3)
- added R9: 470, Resistor_SMD:R_0402_1005Metric, F.Cu at (171.2, 27.4)
- added SW1: SW_Push, Button_Switch_SMD:SW_Push_SPST_NO_Alps_SKRK, F.Cu at (133.0, 80.0)
- added SW2: SW_Push, Button_Switch_SMD:SW_Push_SPST_NO_Alps_SKRK, F.Cu at (136.0, 87.0)
- added SW3: Vin_Switch, Buggy_Footprints:switch123, F.Cu at (66.0, 90.3)
- added U1: USBLC6-2SC6, Package_TO_SOT_SMD:SOT-23-6, F.Cu at (179.0, 35.8)
- added U2: W25Q128JVS, Package_SO:SOIC-8_5.23x5.23mm_P1.27mm, F.Cu at (180.9, 77.2)
- added U3: SOT23-5 200mA 3.3V, Package_TO_SOT_SMD:SOT-23-5, F.Cu at (187.1, 40.1)
- added U4: TP4056, Package_SO:SOP-8-1EP_4.57x4.57mm_P1.27mm_EP4.57x4.45mm, F.Cu at (170.7, 34.2)
- added U5: RP2040, Package_DFN_QFN:QFN-56-1EP_7x7mm_P0.4mm_EP3.2x3.2mm, F.Cu at (179.0, 63.2)
- added Y1: Crystal_GND23, Crystal:Crystal_SMD_3225-4Pin_3.2x2.5mm, F.Cu at (183.2, 69.7)
Routing:
- net +5V: track 0.00 -> 70.7 mm, vias 0 -> 5
- net USB_D+: track 0.00 -> 38.8 mm, vias 0 -> 2
- net USB_D-: track 0.00 -> 38.7 mm, vias 0 -> 2
- net Earth: track 0.00 -> 31.9 mm
- net Charge: track 0.00 -> 30.5 mm, vias 0 -> 1
- net GNDPWR: track 0.00 -> 21.2 mm
- net VBUS: track 0.00 -> 16.4 mm
- net Net-(R11-Pad1): track 0.00 -> 8.84 mm, vias 0 -> 2
- net D-: track 0.00 -> 8.70 mm, vias 0 -> 2
- net D+: track 0.00 -> 8.53 mm, vias 0 -> 2
- net Net-(R10-Pad1): track 0.00 -> 2.96 mm
- net /CC1: track 0.00 -> 2.76 mm
- net /CC2: track 0.00 -> 2.56 mm
- net Net-(D4-Pad2): track 0.00 -> 2.01 mm
- net /VSRC: track 0.00 -> 2.00 mm
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Other:
- board outline added: 24 x 50 mm
