File: RP2040_DevBoard_LiPo_old.kicad_sch (KiCad schematic)
At the start: 52 parts, among them J1 HRO_TYPE-C-31-M-14, J2 Conn_01x16, J3 Battery, J4 Conn_01x18, J5 Conn_01x18, J6 Conn_01x12, Q1 SI2301A, SW1 SW_Push, U1 USBLC6-2SC6, U2 SOT23-5 200mA 3.3V, U3 TP4054, U4 RP2040, U5 W25Q128JVS, Y1 Crystal_GND23

Commit message: Finished routing Featherboard
Parts:
- removed C2, C6: 10uF, Capacitor_SMD:C_0402_1005Metric, symbol Device:C
- removed D1, D3: LED, LED_SMD:LED_1206_3216Metric, symbol Device:LED
- removed J2: Conn_01x16, Connector_PinSocket_2.54mm:PinSocket_1x16_P2.54mm_Vertical, symbol Connector_Generic:Conn_01x16
- removed J3: Battery, Connector_JST:JST_EH_S2B-EH_1x02_P2.50mm_Horizontal, symbol Connector_Generic:Conn_01x02
- removed J6: Conn_01x12, Connector_PinSocket_2.54mm:PinSocket_1x12_P2.54mm_Vertical, symbol Connector_Generic:Conn_01x12
- removed R3: 470, Resistor_SMD:R_0402_1005Metric, symbol Device:R
- removed R4, R5: 10k, Resistor_SMD:R_0402_1005Metric, symbol Device:R
- removed R6: 2k, Resistor_SMD:R_0402_1005Metric, symbol Device:R
- removed SW?: SW_Push, Button_Switch_SMD:SW_Push_SPST_NO_Alps_SKRK, symbol Switch:SW_Push
- removed U3: TP4054, Package_TO_SOT_SMD:SOT-23-5, symbol Battery_Management:MCP73831-2-OT
- added C1: 100nF, Capacitor_SMD:C_0402_1005Metric, symbol Device:C
- added C7, C9: 10 uF, Capacitor_SMD:CP_Elec_3x5.3, symbol Device:C_Polarized_Small
- added C8: 4.7 uF, Capacitor_SMD:C_0402_1005Metric, symbol Device:C_Small
- added D1: BSD3C051V, Diode_SMD:D_SOD-323, symbol Device:D_TVS
- added D4: LED, LED_SMD:LED_1206_3216Metric, symbol Device:LED
- added J4: Battery, Connector_JST:JST_EH_S2B-EH_1x02_P2.50mm_Horizontal, symbol Connector_Generic:Conn_01x02
- added J5: Conn_01x09, Connector_PinSocket_2.54mm:PinSocket_1x09_P2.54mm_Vertical, symbol Connector_Generic:Conn_01x09
- added J7: Conn_01x16, Connector_PinSocket_2.54mm:PinSocket_1x16_P2.54mm_Vertical, symbol Connector_Generic:Conn_01x16
- added L1: BLM15PX121SN1D, Inductor_SMD:L_0402_1005Metric, symbol Device:L_Small
- added R1: 1 MOhm, Resistor_SMD:R_0402_1005Metric, symbol Device:R_Small
- added R10: 1.5k, Resistor_SMD:R_0402_1005Metric, symbol Device:R
- added R11: 5k, Resistor_SMD:R_0603_1608Metric, symbol Device:R_Small
- added R8: 10k, Resistor_SMD:R_0402_1005Metric, symbol Device:R
- added R9: 470, Resistor_SMD:R_0402_1005Metric, symbol Device:R
- added SW2: SW_Push, Button_Switch_SMD:SW_Push_SPST_NO_Alps_SKRK, symbol Switch:SW_Push
- added SW3: Vin_Switch, Buggy_Footprints:switch123, symbol Switch:SW_SPDT
- added U4: TP4056, Package_SO:SOP-8-1EP_4.57x4.57mm_P1.27mm_EP4.57x4.45mm, symbol marbastlib-various:TP4056
- C4: renamed from C3; value 1uF -> 1u
- Q1: value SI2301A -> DMP2045U
- R13: renamed from R9; value 27R -> 27
- R14: renamed from R10; value 27R -> 27
- R7: value 1k -> 1.5k; LCSC C106235 -> C114759
- SW1: LCSC C720477 -> (none)
- U3: renamed from U2; alt1 C9055 -> (none); alt2 C82942 -> (none)
- renumbered C7 to C10, C8 to C11, C10 to C12, C11 to C13, C12 to C14, C13 to C15, C14 to C16, C15 to C17, C16 to C18, C17 to C19, C1 to C2, C18 to C20, C19 to C21, C20 to C22, C9 to C3, C4 to C5, C5 to C6, D2 to D3, J4 to J2, J5 to J3, L1 to L2, R8 to R12, R1 to R2, R2 to R3, R11 to R5, R12 to R6, U5 to U2, U4 to U5
Connections:
- net +3V3: now also J7.16 (Pin_16)
- net +5V: now also R7.2, C7.1, C8.1, R9.2, U4.4 (VCC), U4.8 (CE)
- net +BATT: now also C9.1, J4.1 (Pin_1), SW3.1 (A), SW3.2 (B), U4.5 (BAT)
- net ENABLE: now also R8.2
- net GND: now also R7.1, C7.2, C8.2, C9.2, D1.2 (A2), J4.2 (Pin_2), J5.1 (Pin_1), J7.1 (Pin_1), L1.2, R11.2, SW2.1, U4.1 (TEMP), U4.3 (GND); no longer J1.A1 (GND), J1.A12 (GND), J1.B1 (GND), J1.B12 (GND), R2.2, R3.2
- net GPIO10: now also J5.4 (Pin_4)
- net GPIO11: now also J5.5 (Pin_5)
- net GPIO12: now also J5.6 (Pin_6)
- net GPIO13: now also J5.7 (Pin_7)
- net GPIO14: now also J5.8 (Pin_8)
- net GPIO15: now also J5.9 (Pin_9)
- net GPIO18: now also J7.4 (Pin_4)
- net GPIO19: now also J7.5 (Pin_5)
- net GPIO20: now also J7.6 (Pin_6)
- net GPIO21: now also J7.7 (Pin_7)
- net GPIO22: now also J7.8 (Pin_8)
- net GPIO23: now also J7.9 (Pin_9)
- net GPIO24: now also J7.10 (Pin_10)
- net GPIO25: now also J7.11 (Pin_11)
- net GPIO26: now also J7.12 (Pin_12)
- net GPIO27: now also J7.13 (Pin_13)
- net GPIO28: now also J7.14 (Pin_14)
- net GPIO29: now also J7.15 (Pin_15)
- net GPIO8: now also J5.2 (Pin_2)
- net GPIO9: now also J5.3 (Pin_3)
- net RESET: now also SW2.2
- net SWCLK: now also J7.2 (Pin_2)
- net SWD: now also J7.3 (Pin_3)
- net VSRC: now also R8.1
- net Earth: now reaches J1.S1 (SHIELD)
- net Earth: now also C1.1, R1.1
- new net: R11.1, U4.2 (PROG)
- new net: R10.1, U4.7 (CHRG)
- new net: D4.1 (K), R10.2
- new net: D4.2 (A), R9.1
- new net GNDPWR: C1.2, D1.1 (A1), J1.A1 (GND), J1.A12 (GND), J1.B1 (GND), J1.B12 (GND), L1.1, R1.2, R2.2, R3.2
- no-connect marks 3 -> 4
Other:
- moved on the sheet: C10, C11, C12, C13, C14, C15, C16, C17, C18, C19, C2, C20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
