File: RP2040_DevBoard_LiPo.kicad_sch (KiCad schematic)
At the start: 52 parts, among them J1 HRO_TYPE-C-31-M-14, J2 Conn_01x16, J3 Battery, J4 Conn_01x18, J5 Conn_01x18, J6 Conn_01x12, Q1 SI2301A, SW1 SW_Push, U1 USBLC6-2SC6, U2 SOT23-5 200mA 3.3V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

Commit message: added adjustments to vias around the board
Parts:
- gave numbers to parts that had none: 1
Changed lines of the file:
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@@
   (symbol (lib_id "Switch:SW_Push") (at 71.12 209.55 0) (unit 1)
     (in_bom yes) (on_board yes) (fields_autoplaced)
-    (property "Reference" "SW?" (id 0) (at 71.12 201.93 0))
+    (property "Reference" "SW2" (id 0) (at 71.12 201.93 0))
     (property "Value" "SW_Push" (id 1) (at 71.12 204.47 0))
     (property "Footprint" "Button_Switch_SMD:SW_Push_SPST_NO_Alps_SKRK" (id 2) (at 71.12 204.47 0)
@@
     )
     (path "/73779407-48dd-452b-a964-c307362407a1"
-      (reference "SW?") (unit 1) (value "SW_Push") (footprint "Button_Switch_SMD:SW_Push_SPST_NO_Alps_SKRK")
+      (reference "SW2") (unit 1) (value "SW_Push") (footprint "Button_Switch_SMD:SW_Push_SPST_NO_Alps_SKRK")
     )
     (path "/7e2e56f4-3623-47ac-b08f-ab902d54aa17"
